File: fpvlaptracker32/schematics/fpvlaptracker32.kicad_pcb (KiCad board)
At the start: 2 copper layers, 49 x 49.9 mm, 27 parts, among them J1 Screw_Terminal_01x03, J2 Serial, SW1 Webupdate, SW2 Prog, SW3 Reset, U1 RX5808, U2 LM1117-3.3, U3 ESP-32_WROOM32

Commit message: added files
Parts:
- D5: moved to F.Cu
- moved D5 3.38 mm to (178.7, 100.7), turned to 270 degrees
Routing:
- net +3V3: track 125.1 -> 136.2 mm
- net Net-(D5-Pad1): track 8.38 -> 5.43 mm, vias 1 -> 0
Other:
- board text added: "v1.1"
- board text removed: "v1.0"
Changed lines of the file:
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@@
     (thickness 1.6)
     (drawings 8)
-    (tracks 219)
+    (tracks 221)
     (zones 0)
     (modules 27)
@@
       (net 1 GND))
     (pad 39 smd rect (at 0.3 -2.45 270) (size 6 6) (layers F.Cu F.Paste F.Mask))
+    (model /home/tobi/kicad/libs/kicad-ESP8266/ESP8266.3dshapes/ESP-12E.wrl
+      (offset (xyz 9 -6 0))
+      (scale (xyz 0.5 0.5 0.5))
+      (rotate (xyz 0 0 180))
+    )
   )
   (module LED_SMD:LED_1206_3216Metric_Pad1.42x1.75mm_HandSolder (layer F.Cu)
@@
     )
   )
-  (module LED_SMD:LED_1206_3216Metric_Pad1.42x1.75mm_HandSolder (layer B.Cu)
-    (at 176.7125 98)
+  (module LED_SMD:LED_1206_3216Metric_Pad1.42x1.75mm_HandSolder (layer F.Cu)
+    (at 178.7 100.7375 270)
     (descr "LED SMD 1206 (3216 Metric), square (rectangular) end terminal, IPC_7351 nominal, (Body size source: http://www.tortai-tech.com/upload/download/2011102023233369053.pdf), generated with kicad-footprint-generator")
     (tags "LED handsolder")
     (attr smd)
-    (fp_text reference D5 (at 0 1.82) (layer B.SilkS)
-      (effects (font (size 1 1) (thickness 0.15)) (justify mirror))
-    )
-    (fp_text value LED (at 0 -1.82) (layer B.Fab)
-      (effects (font (size 1 1) (thickness 0.15)) (justify mirror))
-    )
-    (fp_line (start 1.6 0.8) (end -1.2 0.8) (layer B.Fab) (width 0.1))
-    (fp_line (start -1.2 0.8) (end -1.6 0.4) (layer B.Fab) (width 0.1))
-    (fp_line (start -1.6 0.4) (end -1.6 -0.8) (layer B.Fab) (width 0.1))
-    (fp_line (start -1.6 -0.8) (end 1.6 -0.8) (layer B.Fab) (width 0.1))
-    (fp_line (start 1.6 -0.8) (end 1.6 0.8) (layer B.Fab) (width 0.1))
-    (fp_line (start 1.6 1.135) (end -2.46 1.135) (layer B.SilkS) (width 0.12))
-    (fp_line (start -2.46 1.135) (end -2.46 -1.135) (layer B.SilkS) (width 0.12))
-    (fp_line (start -2.46 -1.135) (end 1.6 -1.135) (layer B.SilkS) (width 0.12))
-    (fp_line (start -2.45 -1.12) (end -2.45 1.12) (layer B.CrtYd) (width 0.05))
-    (fp_line (start -2.45 1.12) (end 2.45 1.12) (layer B.CrtYd) (width 0.05))
-    (fp_line (start 2.45 1.12) (end 2.45 -1.12) (layer B.CrtYd) (width 0.05))
-    (fp_line (start 2.45 -1.12) (end -2.45 -1.12) (layer B.CrtYd) (width 0.05))
-    (fp_text user %R (at 0 0) (layer B.Fab)
-      (effects (font (size 0.8 0.8) (thickness 0.12)) (justify mirror))
-    )
-    (pad 1 smd roundrect (at -1.4875 0) (size 1.425 1.75) (layers B.Cu B.Paste B.Mask) (roundrect_rratio 0.175439)
+    (fp_text reference D5 (at 0 -1.82 270) (layer F.SilkS)
+      (effects (font (size 1 1) (thickness 0.15)))
+    )
+    (fp_text value LED (at 0 1.82 270) (layer F.Fab)
+      (effects (font (size 1 1) (thickness 0.15)))
+    )
+    (fp_line (start 1.6 -0.8) (end -1.2 -0.8) (layer F.Fab) (width 0.1))
+    (fp_line (start -1.2 -0.8) (end -1.6 -0.4) (layer F.Fab) (width 0.1))
+    (fp_line (start -1.6 -0.4) (end -1.6 0.8) (layer F.Fab) (width 0.1))
+    (fp_line (start -1.6 0.8) (end 1.6 0.8) (layer F.Fab) (width 0.1))
+    (fp_line (start 1.6 0.8) (end 1.6 -0.8) (layer F.Fab) (width 0.1))
+    (fp_line (start 1.6 -1.135) (end -2.46 -1.135) (layer F.SilkS) (width 0.12))
+    (fp_line (start -2.46 -1.135) (end -2.46 1.135) (layer F.SilkS) (width 0.12))
+    (fp_line (start -2.46 1.135) (end 1.6 1.135) (layer F.SilkS) (width 0.12))
+    (fp_line (start -2.45 1.12) (end -2.45 -1.12) (layer F.CrtYd) (width 0.05))
+    (fp_line (start -2.45 -1.12) (end 2.45 -1.12) (layer F.CrtYd) (width 0.05))
+    (fp_line (start 2.45 -1.12) (end 2.45 1.12) (layer F.CrtYd) (width 0.05))
+    (fp_line (start 2.45 1.12) (end -2.45 1.12) (layer F.CrtYd) (width 0.05))
+    (fp_text user %R (at 0 0 270) (layer F.Fab)
+      (effects (font (size 0.8 0.8) (thickness 0.12)))
+    )
+    (pad 1 smd roundrect (at -1.4875 0 270) (size 1.425 1.75) (layers F.Cu F.Paste F.Mask) (roundrect_rratio 0.175439)
       (net 42 "Net-(D5-Pad1)"))
-    (pad 2 smd roundrect (at 1.4875 0) (size 1.425 1.75) (layers B.Cu B.Paste B.Mask) (roundrect_rratio 0.175439)
+    (pad 2 smd roundrect (at 1.4875 0 270) (size 1.425 1.75) (layers F.Cu F.Paste F.Mask) (roundrect_rratio 0.175439)
       (net 2 +3V3))
     (model ${KISYS3DMOD}/LED_SMD.3dshapes/LED_1206_3216Metric.wrl
@@
     )
   )
-  (gr_text v1.0 (at 149.86 80.01) (layer F.Cu)
+  (gr_text v1.1 (at 149.86 80.01) (layer F.Cu)
     (effects (font (size 1.5 1.5) (thickness 0.3)))
   )
@@
   (via (at 140.97 115.25) (size 0.8) (drill 0.4) (layers F.Cu B.Cu) (net 2))
   (segment (start 173.532 91.44) (end 169.418 91.44) (width 0.499999) (layer B.Cu) (net 2))
-  (segment (start 178.2 97.136) (end 178.2 98) (width 0.499999) (layer B.Cu) (net 2))
-  (segment (start 178.308 97.028) (end 178.2 97.136) (width 0.499999) (layer B.Cu) (net 2))
   (segment (start 173.532 91.44) (end 176.022 91.44) (width 0.499999) (layer B.Cu) (net 2))
-  (segment (start 176.784 95.504) (end 178.308 97.028) (width 0.499999) (layer B.Cu) (net 2))
   (segment (start 176.022 91.44) (end 176.784 92.202) (width 0.499999) (layer B.Cu) (net 2))
   (segment (start 176.784 92.202) (end 176.784 95.504) (width 0.499999) (layer B.Cu) (net 2))
@@
   (segment (start 137.19 115.25) (end 140.75 115.25) (width 0.499999) (layer B.Cu) (net 2))
   (segment (start 167.62 109.75) (end 168.12 110.25) (width 0.499999) (layer F.Cu) (net 2))
-  (segment (start 167.62 100.38) (end 167.62 109.75) (width 0.499999) (layer F.Cu) (net 2))
   (segment (start 168.12 110.25) (end 169.75 110.25) (width 0.499999) (layer F.Cu) (net 2))
   (segment (start 142.05 112.21) (end 142.05 99.65) (width 0.499999) (layer F.Cu) (net 2))
@@
   (segment (start 146.45 122.15) (end 146.45 123.6) (width 0.499999) (layer B.Cu) (net 2))
   (segment (start 145.65 121.35) (end 146.45 122.15) (width 0.499999) (layer B.Cu) (net 2))
-  (segment (start 137.2 119.65) (end 137.25 119.6) (width 0.499999) (layer B.Cu) (net 17))
+  (segment (start 170.25 97.75) (end 170.18 97.82) (width 0.499999) (layer F.Cu) (net 2))
+  (segment (start 167.62 104.35) (end 167.62 104.37) (width 0.499999) (layer F.Cu) (net 2))
+  (segment (start 167.62 100.38) (end 167.62 104.35) (width 0.499999) (layer F.Cu) (net 2))
+  (segment (start 167.62 104.35) (end 167.62 109.75) (width 0.499999) (layer F.Cu) (net 2))
+  (segment (start 167.62 104.37) (end 168.5 105.25) (width 0.499999) (layer F.Cu) (net 2))
+  (segment (start 168.5 105.25) (end 178.05 105.25) (width 0.499999) (layer F.Cu) (net 2))
+  (segment (start 178.7 104.6) (end 178.7 102.225) (width 0.499999) (layer F.Cu) (net 2))
+  (segment (start 178.05 105.25) (end 178.7 104.6) (width 0.499999) (layer F.Cu) (net 2))
   (segment (start 171.836 116.164) (end 177.37 116.164) (width 0.25) (layer B.Cu) (net 3))
   (segment (start 171 117) (end 171.836 116.164) (width 0.25) (layer B.Cu) (net 3))
@@
   (segment (start 152.475 116.225) (end 151 114.75) (width 0.25) (layer F.Cu) (net 14))
   (segment (start 151 114.75) (end 151 113.77) (width 0.25) (layer F.Cu) (net 14))
+  (segment (start 137.2 119.65) (end 137.25 119.6) (width 0.499999) (layer B.Cu) (net 17))
   (segment (start 146.8 116) (end 146.8 118.4) (width 0.25) (layer B.Cu) (net 17))
   (segment (start 145.9 119.3) (end 143.7 119.3) (width 0.25) (layer B.Cu) (net 17))
@@
   (segment (start 160.75 94.8125) (end 160.75 94) (width 0.25) (layer F.Cu) (net 41))
   (segment (start 158.78 97.495) (end 159.58 97.495) (width 0.25) (layer F.Cu) (net 41))
-  (segment (start 178.2 95.975) (end 176.784 97.391) (width 0.25) (layer F.Cu) (net 42))
   (segment (start 178.2 95) (end 178.2 95.975) (width 0.25) (layer F.Cu) (net 42))
-  (via (at 176.784 100.076) (size 0.8) (drill 0.4) (layers F.Cu B.Cu) (net 42))
-  (segment (start 176.784 97.391) (end 176.784 100.076) (width 0.25) (layer F.Cu) (net 42))
-  (segment (start 175.225 98.517) (end 175.225 98) (width 0.25) (layer B.Cu) (net 42))
-  (segment (start 176.784 100.076) (end 175.225 98.517) (width 0.25) (layer B.Cu) (net 42))
+  (segment (start 178.2 95) (end 178.2 96.225) (width 0.25) (layer F.Cu) (net 42))
+  (segment (start 178.7 96.725) (end 178.7 99.25) (width 0.25) (layer F.Cu) (net 42))
+  (segment (start 178.2 96.225) (end 178.7 96.725) (width 0.25) (layer F.Cu) (net 42))
   (zone (net 1) (net_name GND) (layer B.Cu) (hatch edge 0.508)
     (connect_pads (clearance 0.508))

Commit message: updated rev1.1
Parts:
- added J3: Conn_01x01_Female, Connector_PinHeader_2.54mm:PinHeader_1x01_P2.54mm_Vertical, F.Cu at (156.2, 115.2)
- C2, C7, C8, C9, R4, R7, R8: moved to B.Cu
- R5: value 1k -> 100
- R6: value 1k -> 10k; moved to B.Cu
- R9: value 10k -> 1k; moved to B.Cu
- SW1, SW2, SW3: footprint Button_Switch_THT:SW_PUSH_6mm -> Button_Switch_SMD:SW_SPST_KMR2
- U1: moved to F.Cu
- moved D1 40.7 mm to (140.0, 84.2), turned to 270 degrees
- moved R1 40.2 mm to (149.8, 79.0), turned to 180 degrees
- moved D5 39.1 mm to (143.2, 84.2)
- moved R5 32.3 mm to (146.2, 84.2), turned to 270 degrees
- moved SW3 29.1 mm to (142.0, 116.2), turned to 0 degrees
- moved C9 25.6 mm to (140.5, 98.5)
- moved U2 20.8 mm to (158.2, 81.9), turned to 90 degrees
- moved R7 18.3 mm to (145.3, 121.0), turned to 180 degrees
- moved R9 17.8 mm to (145.5, 104.5), turned to 90 degrees
- moved R8 15.4 mm to (150.5, 104.5), turned to 270 degrees
- moved SW1 12.7 mm to (149.5, 116.0)
- moved D4 12.3 mm to (157.2, 88.5), turned to 180 degrees
- moved C8 12.1 mm to (155.2, 95.5), turned to 270 degrees
- moved R6 11.8 mm to (151.5, 121.0)
- moved U1 10.5 mm to (170.8, 105.8), turned to 90 degrees
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Connections:
- U3 pad 12: Net-(U3-Pad12) -> /ADC_REF
Routing:
- net +3V3: track 136.2 -> 83.5 mm
- net /EN: track 41.9 -> 13.6 mm, vias 2 -> 1
- net /LED: track 34.2 -> 6.53 mm, vias 2 -> 0
- net /RSSI: track 16.7 -> 42.9 mm
- net +5V: track 60.0 -> 44.4 mm, vias 3 -> 1
- net /ANALOG_RSSI: track 29.6 -> 14.2 mm
- net /BAT: track 34.4 -> 44.7 mm
- net /WEB_UPDATE: track 22.8 -> 13.8 mm, vias 0 -> 1
- net /ADC_REF: track 0.00 -> 8.13 mm
- net Net-(D1-Pad1): track 2.76 -> 10.4 mm
- net /SPI_DATA: track 36.5 -> 43.6 mm, vias 3 -> 0
- net /ANALOG_BAT: track 21.2 -> 14.8 mm, vias 0 -> 1
- net /IO0: track 13.3 -> 16.9 mm, vias 0 -> 2
- net Net-(R4-Pad2): track 4.78 -> 8.15 mm, vias 0 -> 1
- net /RXD: track 16.5 -> 13.9 mm, vias 0 -> 1
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Other:
- board text added: "+5V GND BAT"
- board text added: "FLASH"
- board text added: "OTA"
- board text added: "RESET"
- board text added: "RX TX GND"
- board text added: "VREF"
- board text added: "fpvlaptracker32 v1.1"
- board text removed: "fpvlaptracker32"
- board text removed: "v1.1"
